Commit message: Simple demo system
Should work.

File: tb_robot/robots/m600.xacro (robot description, xacro)
@@ -23,4 +23,7 @@
 	<xacro:velodyne>
 	</xacro:velodyne>
+	<xacro:include filename="$(find tb_robot)/urdf/velodyne_virtuals.urdf.xacro" />
+	<xacro:velodyne_virtuals>
+	</xacro:velodyne_virtuals>
 	<xacro:include filename="$(find tb_robot)/urdf/lidarlite.urdf.xacro" />
 	<xacro:lidarlite>

File: tb_robot/urdf/velodyne.urdf.xacro (robot description, xacro)
@@ -6,6 +6,4 @@
 	  <link name="velodyne"></link>
 	  <link name="velodyne_aligned"></link>
-		<link name="velodyne_up"/>
-		<link name="velodyne_down"/>
 	   <link name="velodyne_link">
 	      <inertial>
@@ -43,14 +41,4 @@
 	           <child link="velodyne_aligned"/>
 	     </joint>
-			 <joint name="velodyne_joint_down" type="fixed" >
-	 					<origin xyz="0 0 3.0" rpy="0 0 0" />
-	 					<parent link="velodyne_aligned" />
-	 					<child link="velodyne_up"/>
-	 			</joint>
-	 		<joint name="velodyne_joint_up" type="fixed" >
-	 					<origin xyz="0 0 -3.0" rpy="0 0 0" />
-	 					<parent link="velodyne_aligned" />
-	 					<child link="velodyne_down"/>
-	 				</joint>
   </xacro:macro>
 </robot>
