Commit message: private_temp2

File: tb_robot/urdf/velodyne_virtuals.urdf.xacro (robot description, xacro)
@@ -8,10 +8,10 @@
  	 <link name="velodyne_tilt_up"></link>
  	 <joint name="velodyne_joint_down" type="fixed" >
- 				<origin xyz="0 0 3.0" rpy="0 0 0" />
+ 				<origin xyz="0 0 1.0" rpy="0 0 0" />
  				<parent link="velodyne_aligned" />
  				<child link="velodyne_up"/>
  		</joint>
  	<joint name="velodyne_joint_up" type="fixed" >
-		<origin xyz="0 0 -3.0" rpy="0 0 0" />
+		<origin xyz="0 0 -1.0" rpy="0 0 0" />
 		<parent link="velodyne_aligned" />
 		<child link="velodyne_down"/>
